File: pcb/pl60c_dmx.kicad_pcb (KiCad board)
At the start: 2 copper layers, 80 x 54 mm, 39 parts, among them J1 USB-C 16P, J2 XLR-5 female (DMX OUT), J3 DMX pigtail, J4 EXPANSION, J5 UART0, Q1 S8050, SW1 RESET, SW2 BOOT, SW3 USER, U1 ESP32-S3-WROOM-1-N8, U2 AMS1117-3.3, U3 MAX3485, U4 USBLC6-2SC6

Commit message: auto: 2026-09-02 13:00:39
Co-Authored-By: Claude Fable 5.1 <noreply@anthropic.com>
Claude-Session: https://claude.ai/code/session_01WsrVZb94LwbHVAmBvsSTfn
Parts:
- moved D3 3.54 mm to (59.5, 37.0)
- moved Q1 3.50 mm to (55.0, 37.0)
- moved R9 3.50 mm to (50.5, 37.0)
- moved BZ1 2.06 mm to (69.0, 41.5)
- moved C6 1.50 mm to (15.0, 42.5)
- moved C8 1.50 mm to (39.0, 43.5)
- moved D2 1.50 mm to (43.5, 48.5)
- moved R3 1.50 mm to (10.5, 42.5)
- moved R4 1.50 mm to (23.5, 42.5)
- moved R5 1.50 mm to (34.5, 42.5)
- moved R8 1.50 mm to (43.5, 43.5)
- moved SW1 1.50 mm to (12.5, 48.0)
- moved SW2 1.50 mm to (23.5, 48.0)
- moved SW3 1.50 mm to (34.5, 48.0)
- moved J1 1.20 mm to (3.10, 31.0), turned to -90 degrees
Routing:
- net +3V3: track 0.00 -> 143.2 mm, vias 0 -> 2
- net DMX_B: track 0.00 -> 66.5 mm, vias 0 -> 2
- net EN: track 0.00 -> 64.9 mm, vias 0 -> 2
- net BTN_USER: track 0.00 -> 59.4 mm, vias 0 -> 2
- net BUZZER: track 0.00 -> 54.7 mm, vias 0 -> 2
- net IO0_BOOT: track 0.00 -> 52.7 mm, vias 0 -> 2
- net DMX_A: track 0.00 -> 50.5 mm, vias 0 -> 1
- net VBUS: track 0.00 -> 41.2 mm, vias 0 -> 3
- net USB_D-: track 0.00 -> 39.4 mm, vias 0 -> 3
- net DMX_DE: track 0.00 -> 36.3 mm, vias 0 -> 2
- net USB_D+: track 0.00 -> 33.0 mm, vias 0 -> 2
- net EXP_SDA: track 0.00 -> 31.8 mm, vias 0 -> 1
- net RXD0: track 0.00 -> 29.0 mm, vias 0 -> 1
- net TXD0: track 0.00 -> 28.6 mm, vias 0 -> 1
- net +5V: track 0.00 -> 28.3 mm, vias 0 -> 4
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
Commit message: auto: 2026-09-02 13:06:45
Co-Authored-By: Claude Fable 5.1 <noreply@anthropic.com>
Claude-Session: https://claude.ai/code/session_01WsrVZb94LwbHVAmBvsSTfn
Parts:
- C6: footprint C_0603_1608Metric -> C_0805_2012Metric
- D1: value SM712 -> PSM712
- D3: value 1N4148W -> B5819W
- F1: value 0.75A PTC -> 1A PTC
- SW1, SW2, SW3: footprint SW_SPST_PTS645Sx43SMTR92 -> SW_SPST_SKQG_WithStem
- U1: value ESP32-S3-WROOM-1-N8 -> ESP32-S3-WROOM-1-N16R8
- U3: value MAX3485 -> SP3485EN
Routing:
- net +3V3: track 143.2 -> 0.00 mm, vias 2 -> 0
- net DMX_B: track 66.5 -> 0.00 mm, vias 2 -> 0
- net EN: track 64.9 -> 0.00 mm, vias 2 -> 0
- net BTN_USER: track 59.4 -> 0.00 mm, vias 2 -> 0
- net BUZZER: track 54.7 -> 0.00 mm, vias 2 -> 0
- net IO0_BOOT: track 52.7 -> 0.00 mm, vias 2 -> 0
- net DMX_A: track 50.5 -> 0.00 mm, vias 1 -> 0
- net VBUS: track 41.2 -> 0.00 mm, vias 3 -> 0
- net USB_D-: track 39.4 -> 0.00 mm, vias 3 -> 0
- net DMX_DE: track 36.3 -> 0.00 mm, vias 2 -> 0
- net GND: track 0.00 -> 34.5 mm, vias 0 -> 59
- net USB_D+: track 33.0 -> 0.00 mm, vias 2 -> 0
- net EXP_SDA: track 31.8 -> 0.00 mm, vias 1 -> 0
- net RXD0: track 29.0 -> 0.00 mm, vias 1 -> 0
- net TXD0: track 28.6 -> 0.00 mm, vias 1 -> 0
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
Commit message: auto: 2026-09-02 13:08:46
Co-Authored-By: Claude Fable 5.1 <noreply@anthropic.com>
Claude-Session: https://claude.ai/code/session_01WsrVZb94LwbHVAmBvsSTfn
Routing:
- net +3V3: track 0.00 -> 156.7 mm, vias 0 -> 2
- net +5V: track 0.00 -> 86.2 mm
- net DMX_B: track 0.00 -> 70.1 mm
- net EN: track 0.00 -> 67.0 mm, vias 0 -> 2
- net BTN_USER: track 0.00 -> 55.7 mm, vias 0 -> 2
- net BUZZER: track 0.00 -> 53.3 mm, vias 0 -> 2
- net DMX_A: track 0.00 -> 52.4 mm
- net DMX_DE: track 0.00 -> 46.3 mm
- net USB_D+: track 0.00 -> 45.9 mm, vias 0 -> 2
- net IO0_BOOT: track 0.00 -> 41.9 mm, vias 0 -> 2
- net VBUS: track 0.00 -> 41.0 mm
- net USB_D-: track 0.00 -> 38.9 mm, vias 0 -> 3
- net GND: track 34.5 -> 0.00 mm, vias 59 -> 0
- net LED_DATA: track 0.00 -> 29.0 mm, vias 0 -> 2
- net EXP_IO11: track 0.00 -> 28.7 mm, vias 0 -> 1
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
Commit message: auto: 2026-09-02 13:10:48
Co-Authored-By: Claude Fable 5.1 <noreply@anthropic.com>
Claude-Session: https://claude.ai/code/session_01WsrVZb94LwbHVAmBvsSTfn
Routing:
- net +3V3: track 156.7 -> 0.00 mm, vias 2 -> 0
- net +5V: track 86.2 -> 0.00 mm
- net DMX_B: track 70.1 -> 0.00 mm
- net EN: track 67.0 -> 0.00 mm, vias 2 -> 0
- net BTN_USER: track 55.7 -> 0.00 mm, vias 2 -> 0
- net BUZZER: track 53.3 -> 0.00 mm, vias 2 -> 0
- net DMX_A: track 52.4 -> 0.00 mm
- net DMX_DE: track 46.3 -> 0.00 mm
- net USB_D+: track 45.9 -> 0.00 mm, vias 2 -> 0
- net GND: track 0.00 -> 44.8 mm, vias 0 -> 129
- net IO0_BOOT: track 41.9 -> 0.00 mm, vias 2 -> 0
- net VBUS: track 41.0 -> 0.00 mm
- net USB_D-: track 38.9 -> 0.00 mm, vias 3 -> 0
- net LED_DATA: track 29.0 -> 0.00 mm, vias 2 -> 0
- net EXP_IO11: track 28.7 -> 0.00 mm, vias 1 -> 0
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
Commit message: auto: 2026-09-02 13:12:50
Co-Authored-By: Claude Fable 5.1 <noreply@anthropic.com>
Claude-Session: https://claude.ai/code/session_01WsrVZb94LwbHVAmBvsSTfn
Routing:
- net +3V3: track 0.00 -> 152.4 mm, vias 0 -> 5
- net +5V: track 0.00 -> 97.2 mm, vias 0 -> 4
- net DMX_A: track 0.00 -> 64.4 mm
- net DMX_B: track 0.00 -> 62.7 mm, vias 0 -> 2
- net EN: track 0.00 -> 60.8 mm, vias 0 -> 2
- net BTN_USER: track 0.00 -> 59.8 mm, vias 0 -> 2
- net IO0_BOOT: track 0.00 -> 57.5 mm, vias 0 -> 2
- net BUZZER: track 0.00 -> 53.2 mm, vias 0 -> 2
- net DMX_DE: track 0.00 -> 33.5 mm, vias 0 -> 2
- net VBUS: track 0.00 -> 33.4 mm, vias 0 -> 2
- net LED_DATA: track 0.00 -> 31.6 mm, vias 0 -> 2
- net EXP_SDA: track 0.00 -> 31.0 mm, vias 0 -> 1
- net TXD0: track 0.00 -> 28.9 mm, vias 0 -> 1
- net EXP_IO11: track 0.00 -> 28.9 mm, vias 0 -> 1
- net RXD0: track 0.00 -> 28.5 mm, vias 0 -> 1
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
Commit message: auto: 2026-09-02 13:14:52
Co-Authored-By: Claude Fable 5.1 <noreply@anthropic.com>
Claude-Session: https://claude.ai/code/session_01WsrVZb94LwbHVAmBvsSTfn
Routing:
- net GND: track 48.7 -> 385.9 mm, vias 127 -> 77
- net +3V3: track 152.4 -> 176.0 mm, vias 5 -> 3
- net CC2: track 0.00 -> 10.4 mm, vias 0 -> 2
- net BZ_N: track 23.7 -> 15.2 mm, vias 0 -> 2
- net +5V: track 97.2 -> 89.5 mm, vias 4 -> 2
- net IO0_BOOT: track 57.5 -> 50.4 mm
- net DMX_A: track 64.4 -> 57.5 mm
- net EN: track 60.8 -> 55.0 mm
- net EXP_IO11: track 28.9 -> 23.6 mm
- net VBUS: track 33.4 -> 37.4 mm
- net BTN_USER: track 59.8 -> 55.8 mm
- net USB_D+: track 24.1 -> 20.3 mm
- net DMX_TX: track 24.7 -> 27.2 mm
- net BUZZER: track 53.2 -> 50.8 mm
- net TXD0: track 28.9 -> 26.6 mm
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
Commit message: auto: 2026-09-02 13:16:54
Co-Authored-By: Claude Fable 5.1 <noreply@anthropic.com>
Claude-Session: https://claude.ai/code/session_01WsrVZb94LwbHVAmBvsSTfn
Parts:
- moved R1 2.06 mm to (14.0, 26.0)
- moved R2 2.06 mm to (14.0, 36.0)
- moved U4 2.00 mm to (16.5, 31.0)
Routing:
- net USB_D+: track 20.3 -> 59.0 mm, vias 2 -> 3
- net +3V3: track 176.0 -> 149.1 mm, vias 3 -> 2
- net GND: track 385.9 -> 360.9 mm, vias 77 -> 76
- net IO0_BOOT: track 50.4 -> 74.2 mm
- net DMX_TX: track 27.2 -> 42.5 mm
- net USB_D-: track 21.8 -> 36.2 mm, vias 2 -> 3
- net CC1: track 0.00 -> 9.78 mm, vias 0 -> 2
- net +5V: track 89.5 -> 99.1 mm, vias 2 -> 0
- net EN: track 55.0 -> 62.5 mm
- net VBUS: track 37.4 -> 42.8 mm, vias 2 -> 3
- net BUZZER: track 50.8 -> 46.6 mm
- net EXP_SDA: track 30.5 -> 26.6 mm
- net DMX_B: track 62.3 -> 59.1 mm
- net DMX_A: track 57.5 -> 54.4 mm
- net LED_DATA: track 29.7 -> 27.6 mm
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
Commit message: auto: 2026-09-02 13:18:56
Co-Authored-By: Claude Fable 5.1 <noreply@anthropic.com>
Claude-Session: https://claude.ai/code/session_01WsrVZb94LwbHVAmBvsSTfn
Routing:
- net +3V3: track 149.1 -> 177.8 mm, vias 2 -> 3
- net IO0_BOOT: track 74.2 -> 48.4 mm
- net USB_D+: track 59.0 -> 41.9 mm, vias 3 -> 4
- net +5V: track 99.1 -> 89.6 mm, vias 0 -> 2
- net USB_D-: track 36.2 -> 27.6 mm, vias 3 -> 2
- net DMX_RX: track 28.0 -> 36.3 mm
- net GND: track 360.9 -> 368.9 mm
- net EN: track 62.5 -> 55.8 mm
- net DMX_B: track 59.1 -> 65.7 mm
- net DMX_TX: track 42.5 -> 38.4 mm
- net EXP_IO11: track 25.1 -> 21.9 mm
- net BTN_USER: track 55.9 -> 58.8 mm
- net VBUS: track 42.8 -> 45.1 mm
- net LED_DATA: track 27.6 -> 29.5 mm
- net CC1: track 9.78 -> 8.08 mm
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