File: pcb/pl60c_dmx.kicad_pcb (KiCad board)
At the start: 2 copper layers, 80 x 54 mm, 40 parts, among them J1 USB-C 16P, J2 XLR-5 female (DMX OUT), J3 DMX pigtail, J4 EXPANSION, J5 UART0, Q1 S8050, SW1 RESET, SW2 BOOT, SW3 USER, U1 ESP32-S3-WROOM-1-N16R8, U2 AMS1117-3.3, U3 SP3485EN, U4 USBLC6-2SC6

Commit message: auto: 2026-09-02 14:56:10
Co-Authored-By: Claude Fable 5.1 <noreply@anthropic.com>
Claude-Session: https://claude.ai/code/session_01WsrVZb94LwbHVAmBvsSTfn
Routing:
- net DMX_DE: track 31.8 -> 47.4 mm
- net DMX_TX: track 28.7 -> 40.0 mm
- net +3V3: track 167.0 -> 156.5 mm, vias 6 -> 4
- net IO0_BOOT: track 47.5 -> 55.0 mm, vias 4 -> 2
- net BUZZER: track 45.4 -> 52.5 mm
- net EXP_IO10: track 31.2 -> 24.7 mm
- net DMX_RX: track 31.7 -> 36.3 mm
- net GND: track 465.8 -> 469.8 mm
- net EXP_SDA: track 30.1 -> 26.7 mm
- net EXP_IO11: track 28.6 -> 25.4 mm
- net BZ_P: track 22.8 -> 19.7 mm
- net USB_D+: track 42.1 -> 39.3 mm, vias 4 -> 5
- net VBUS: track 46.1 -> 48.4 mm
- net EN: track 63.9 -> 62.0 mm
- net EXP_SCL: track 22.4 -> 24.2 mm, vias 0 -> 1
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