File: pcb/pl60c_dmx_mini.kicad_pcb (KiCad board)
At the start: 4 copper layers, 38.5 x 28.5 mm, 35 parts, among them J1 USB-C 16P, J2 XLR-5 female (DMX OUT), Q1 S8050, SW2 BOOT, SW3 USER, U1 ESP32-S3-MINI-1-N8, U2 AP2112K-3.3, U3 SP3485EN, U4 USBLC6-2SC6

Commit message: auto: 2026-09-02 14:14:01
Co-Authored-By: Claude Fable 5.1 <noreply@anthropic.com>
Claude-Session: https://claude.ai/code/session_01WsrVZb94LwbHVAmBvsSTfn
Parts:
- removed BZ1: MLT-8530, MagneticBuzzer_CUI_CMT-8504-100-SMT
- added TP5: BZ+, TestPoint_Pad_1.5x1.5mm, B.Cu at (28.5, 28.0)
- added TP6: BZ-, TestPoint_Pad_1.5x1.5mm, B.Cu at (31.2, 28.0)
- moved C6 8.29 mm to (3.50, 12.0)
- moved R3 8.15 mm to (3.50, 10.0)
- moved C5 8.04 mm to (3.50, 8.00)
- moved R4 5.75 mm to (6.50, 8.00)
- moved R5 5.50 mm to (6.50, 10.0)
- moved R8 5.29 mm to (6.50, 12.0)
- moved C8 4.75 mm to (9.50, 12.0)
- moved R9 0.96 mm to (6.00, 2.50)
- moved Q1 0.71 mm to (3.00, 4.00)
- moved U1 0.70 mm to (5.25, 9.50)
- moved C1 0.50 mm to (3.00, 19.8)
- moved C2 0.50 mm to (14.5, 25.3)
- moved C3 0.50 mm to (10.6, 20.3)
- moved D1 0.50 mm to (17.9, 19.4)
- moved D3 0.50 mm to (8.50, 4.50)
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Routing:
- net GND: track 64.5 -> 69.1 mm, vias 50 -> 56
- net USB_D-: track 7.50 -> 5.90 mm
- net USB_D+: track 12.8 -> 11.3 mm
- added copper zone on In2.Cu, net GND
- removed copper zone on In2.Cu, net +3V3
Other:
- board size 38.5 x 28.5 mm -> 38.5 x 29 mm
- board text added: "BZ+ BZ-"

Commit message: auto: 2026-09-02 14:16:03
Co-Authored-By: Claude Fable 5.1 <noreply@anthropic.com>
Claude-Session: https://claude.ai/code/session_01WsrVZb94LwbHVAmBvsSTfn
Parts:
- moved C3 8.12 mm to (17.0, 25.3), turned to 0 degrees
- moved C1 7.73 mm to (10.6, 18.4)
- moved R4 4.80 mm to (11.3, 8.00)
- moved R5 4.80 mm to (11.3, 10.0)
- moved R8 4.80 mm to (11.3, 12.0)
- moved C8 1.50 mm to (9.50, 13.5)
- moved TP5 0.50 mm to (28.5, 27.5)
- moved TP6 0.50 mm to (31.2, 27.5)
Routing:
- net GND: track 69.1 -> 71.6 mm, vias 56 -> 58

Commit message: auto: 2026-09-02 14:18:05
Co-Authored-By: Claude Fable 5.1 <noreply@anthropic.com>
Claude-Session: https://claude.ai/code/session_01WsrVZb94LwbHVAmBvsSTfn
Parts:
- moved TP5 9.30 mm to (34.0, 20.0)
- moved TP6 9.24 mm to (36.6, 20.0)
Routing:
- net USB_D+: track 11.3 -> 10.1 mm
- net USB_D-: track 5.90 -> 5.30 mm

Commit message: auto: 2026-09-02 14:20:07
Co-Authored-By: Claude Fable 5.1 <noreply@anthropic.com>
Claude-Session: https://claude.ai/code/session_01WsrVZb94LwbHVAmBvsSTfn
Routing:
- net +3V3: track 0.00 -> 97.9 mm, vias 0 -> 5
- net +5V: track 0.00 -> 53.0 mm, vias 0 -> 2
- net BZ_N: track 0.00 -> 48.5 mm, vias 0 -> 2
- net EXP_SCL: track 0.00 -> 29.3 mm, vias 0 -> 1
- net EXP_SDA: track 0.00 -> 27.5 mm, vias 0 -> 1
- net DMX_B: track 0.00 -> 27.2 mm
- net IO0_BOOT: track 0.00 -> 26.8 mm, vias 0 -> 3
- net USB_D+: track 10.1 -> 35.8 mm, vias 2 -> 4
- net BTN_USER: track 0.00 -> 23.7 mm, vias 0 -> 3
- net DMX_A: track 0.00 -> 22.5 mm, vias 0 -> 1
- net BUZZER: track 0.00 -> 16.5 mm, vias 0 -> 2
- net LED_DATA_R: track 0.00 -> 16.2 mm, vias 0 -> 2
- net GND: track 71.6 -> 86.5 mm
- net EN: track 0.00 -> 12.4 mm, vias 0 -> 2
- net LED_DATA: track 0.00 -> 11.5 mm, vias 0 -> 2
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
Commit message: auto: 2026-09-02 14:22:09
Co-Authored-By: Claude Fable 5.1 <noreply@anthropic.com>
Claude-Session: https://claude.ai/code/session_01WsrVZb94LwbHVAmBvsSTfn
Parts:
- moved TP6 34.0 mm to (3.00, 15.0)
- moved TP5 28.4 mm to (6.00, 15.0)
Routing:
- net BZ_N: track 48.5 -> 7.14 mm, vias 2 -> 0
- net +5V: track 53.0 -> 30.4 mm, vias 2 -> 0
- net USB_D-: track 7.58 -> 29.1 mm, vias 0 -> 3
- net LED_DATA: track 11.5 -> 22.8 mm
- net DMX_B: track 27.2 -> 36.0 mm
- net USB_D+: track 35.8 -> 40.4 mm, vias 4 -> 3
- net DMX_TX: track 3.43 -> 7.93 mm
- net DMX_A: track 22.5 -> 18.3 mm, vias 1 -> 0
- net BUZZER: track 16.5 -> 20.6 mm
- net BTN_USER: track 23.7 -> 27.5 mm, vias 3 -> 2
- net Q1_B: track 8.40 -> 4.74 mm
- net EN: track 12.4 -> 15.4 mm
- net VBUS: track 17.5 -> 20.3 mm
- net IO0_BOOT: track 26.8 -> 28.8 mm, vias 3 -> 2
- net CC2: track 8.82 -> 6.80 mm
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Other:
- board text added: "BZ- BZ+"
- board text removed: "BZ+ BZ-"

Commit message: auto: 2026-09-02 14:24:11
Co-Authored-By: Claude Fable 5.1 <noreply@anthropic.com>
Claude-Session: https://claude.ai/code/session_01WsrVZb94LwbHVAmBvsSTfn
Routing:
- net BZ_N: track 7.14 -> 19.6 mm, vias 0 -> 2
- net LED_DATA_R: track 15.1 -> 26.6 mm
- net LED_DATA: track 22.8 -> 11.3 mm, vias 2 -> 1
- net VBUS: track 20.3 -> 31.4 mm, vias 3 -> 4
- net USB_D-: track 29.1 -> 39.5 mm
- net USB_D+: track 40.4 -> 33.0 mm
- net +3V3: track 97.0 -> 104.3 mm
- net DMX_TX: track 7.93 -> 3.01 mm
- net IO0_BOOT: track 28.8 -> 32.9 mm
- net EN: track 15.4 -> 12.1 mm
- net CC1: track 10.2 -> 7.28 mm
- net Q1_B: track 4.74 -> 7.02 mm
- net BUZZER: track 20.6 -> 21.0 mm, vias 2 -> 1
- net BTN_USER: track 27.5 -> 27.6 mm, vias 2 -> 3

Commit message: auto: 2026-09-02 14:26:12
Co-Authored-By: Claude Fable 5.1 <noreply@anthropic.com>
Claude-Session: https://claude.ai/code/session_01WsrVZb94LwbHVAmBvsSTfn
Routing:
- net USB_D+: track 33.0 -> 48.2 mm
- net BUZZER: track 21.0 -> 29.5 mm, vias 1 -> 2
- net VBUS: track 31.4 -> 25.7 mm, vias 4 -> 3
- net DMX_B: track 36.0 -> 31.0 mm
- net LED_DATA_R: track 26.6 -> 22.1 mm
- net BTN_USER: track 27.6 -> 23.5 mm, vias 3 -> 2
- net EN: track 12.1 -> 15.8 mm, vias 2 -> 1
- net BZ_N: track 19.6 -> 21.9 mm, vias 2 -> 0
- net +5V: track 30.5 -> 32.8 mm, vias 0 -> 2
- net Q1_B: track 7.02 -> 5.21 mm
- net GND: track 85.4 -> 86.3 mm
- net CC2: track 6.72 -> 7.58 mm
- net IO0_BOOT: track 32.9 -> 33.2 mm, vias 2 -> 3
- net LED_DATA: track 11.3 -> 11.4 mm, vias 1 -> 2

Commit message: auto: 2026-09-02 14:45:57
Co-Authored-By: Claude Fable 5.1 <noreply@anthropic.com>
Claude-Session: https://claude.ai/code/session_01WsrVZb94LwbHVAmBvsSTfn
Parts:
- added R10: 10R, R_1206_3216Metric, B.Cu at (12.9, 15.4)
- F1: value 0.75A PTC -> 1A PTC; footprint Fuse_0805_2012Metric -> Fuse_1206_3216Metric
- R9: value 1k -> 470R
- moved C4 15.3 mm to (3.00, 15.0), turned to 90 degrees
- moved C8 10.9 mm to (12.5, 3.00)
- moved TP6 6.20 mm to (9.20, 14.9)
- moved C5 5.39 mm to (1.50, 13.0), turned to 90 degrees
- moved R7 1.63 mm to (16.3, 14.8)
- moved TP5 0.51 mm to (6.50, 14.9)
Connections:
- D3 pad 1: +5V -> BZ_P
- Q1 pad 1: GND -> Q1_B
- Q1 pad 2: Q1_B -> GND
- TP5 pad 1: +5V -> BZ_P
Routing:
- net USB_D-: track 39.8 -> 12.6 mm, vias 3 -> 2
- net BZ_P: track 0.00 -> 22.9 mm, vias 0 -> 2
- net +5V: track 32.8 -> 15.0 mm, vias 2 -> 0
- net USB_D+: track 48.2 -> 31.1 mm
- net +3V3: track 103.9 -> 89.5 mm, vias 4 -> 3
- net VBUS: track 25.7 -> 15.7 mm, vias 3 -> 2
- net LED_DATA_R: track 22.1 -> 13.1 mm
- net BUZZER: track 29.5 -> 22.3 mm
- net DMX_TX: track 3.31 -> 10.2 mm
- net IO0_BOOT: track 33.2 -> 38.5 mm
- net DMX_B: track 31.0 -> 26.5 mm
- net BZ_N: track 21.9 -> 18.5 mm, vias 0 -> 2
- net EXP_SDA: track 27.7 -> 30.3 mm, vias 1 -> 2
- net CC1: track 7.28 -> 9.75 mm, vias 1 -> 2
- net Q1_B: track 5.21 -> 7.34 mm, vias 0 -> 2
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Other:
- board text added: "BZ+ BZ-"
- board text removed: "BZ- BZ+"
