File: pcb/pl60c_dmx_mini.kicad_sch (KiCad schematic)
At the start: 37 parts, among them J1 USB-C 16P, J2 XLR-5 female (DMX OUT), Q1 S8050, SW2 BOOT, SW3 USER, U1 ESP32-S3-MINI-1-N8, U2 AP2112K-3.3, U3 SP3485EN, U4 USBLC6-2SC6

Commit message: auto: 2026-09-02 13:50:15
Co-Authored-By: Claude Fable 5.1 <noreply@anthropic.com>
Claude-Session: https://claude.ai/code/session_01WsrVZb94LwbHVAmBvsSTfn
Parts:
- F1: value 1A PTC -> 0.75A PTC; footprint Fuse:Fuse_1206_3216Metric -> Fuse:Fuse_0805_2012Metric; LCSC C5358568 -> C7472571; MPN BSMD1206-100-30V -> 0805L075/6AR
- U1: LCSC TBD -> C2913206
Changed lines of the file:
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@@
 			)
 		)
-		(property "Value" "1A PTC"
+		(property "Value" "0.75A PTC"
 			(at 69.85 46.99 0)
 			(effects
@@
 			)
 		)
-		(property "Footprint" "Fuse:Fuse_1206_3216Metric"
+		(property "Footprint" "Fuse:Fuse_0805_2012Metric"
 			(at 69.85 39.37 0)
 			(effects
@@
 			)
 		)
-		(property "Description" "PTC resettable fuse 1206, 1 A hold / 1.8 A trip, 30 V"
+		(property "Description" "PTC resettable fuse 0805, 0.75 A hold, 6 V"
 			(at 69.85 39.37 0)
 			(effects
@@
 			)
 		)
-		(property "LCSC" "C5358568"
+		(property "LCSC" "C7472571"
 			(at 69.85 39.37 0)
 			(effects
@@
 			)
 		)
-		(property "MPN" "BSMD1206-100-30V"
+		(property "MPN" "0805L075/6AR"
 			(at 69.85 39.37 0)
 			(effects
@@
 			)
 		)
-		(property "LCSC" "TBD"
+		(property "LCSC" "C2913206"
 			(at 199.39 80.01 0)
 			(effects

Commit message: auto: 2026-09-02 14:02:26
Co-Authored-By: Claude Fable 5.1 <noreply@anthropic.com>
Claude-Session: https://claude.ai/code/session_01WsrVZb94LwbHVAmBvsSTfn
Parts:
- removed TP5: TXD0, TestPoint:TestPoint_Pad_1.5x1.5mm, symbol Connector:TestPoint
- removed TP6: RXD0, TestPoint:TestPoint_Pad_1.5x1.5mm, symbol Connector:TestPoint
Connections:
- net RXD0: no longer names the net of U1.40 (RXD0)
- net TXD0: no longer names the net of U1.39 (TXD0)
- no-connect marks 33 -> 35
Other:
- note added: "Test pads: I2C expansion (RTC / sensor)"
- note removed: "Test pads: I2C expansion and UART0"
Changed lines of the file:
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@@
 		(at 214.63 95.25)
 	)
-	(wire
-		(pts
-			(xy 214.63 54.61)
-			(xy 217.17 54.61)
-		)
-		(stroke
-			(width 0)
-			(type default)
-		)
-	)
-	(label "TXD0"
-		(at 217.17 54.61 0)
-		(fields_autoplaced yes)
-		(effects
-			(font
-				(size 1.27 1.27)
-			)
-			(justify left bottom)
-		)
-	)
-	(wire
-		(pts
-			(xy 214.63 57.15)
-			(xy 217.17 57.15)
-		)
-		(stroke
-			(width 0)
-			(type default)
-		)
+	(no_connect
+		(at 214.63 54.61)
 	)
-	(label "RXD0"
-		(at 217.17 57.15 0)
-		(fields_autoplaced yes)
-		(effects
-			(font
-				(size 1.27 1.27)
-			)
-			(justify left bottom)
-		)
+	(no_connect
+		(at 214.63 57.15)
 	)
 	(no_connect
@@
 		)
 	)
-	(symbol
-		(lib_id "Connector:TestPoint")
-		(at 379.73 190.5 0)
-		(unit 1)
-		(exclude_from_sim no)
-		(in_bom yes)
-		(on_board yes)
-		(dnp no)
-		(property "Reference" "TP5"
-			(at 379.73 186.69 0)
-			(effects
-				(font
-					(size 1.27 1.27)
-				)
-			)
-		)
-		(property "Value" "TXD0"
-			(at 379.73 194.31 0)
-			(effects
-				(font
-					(size 1.27 1.27)
-				)
-			)
-		)
-		(property "Footprint" "TestPoint:TestPoint_Pad_1.5x1.5mm"
-			(at 379.73 190.5 0)
-			(effects
-				(font
-					(size 1.27 1.27)
-				)
-				(hide yes)
-			)
-		)
-		(property "Datasheet" "~"
-			(at 379.73 190.5 0)
-			(effects
-				(font
-					(size 1.27 1.27)
-				)
-				(hide yes)
-			)
-		)
-		(property "Description" "Test pad 1.5 mm"
-			(at 379.73 190.5 0)
-			(effects
-				(font
-					(size 1.27 1.27)
-				)
-				(hide yes)
-			)
-		)
-		(property "LCSC" ""
-			(at 379.73 190.5 0)
-			(effects
-				(font
-					(size 1.27 1.27)
-				)
-				(hide yes)
-			)
-		)
-		(pin "1"
-		)
-		(instances
-			(project "pl60c_dmx_mini"
-				(path "/e63f84e3-7254-5f79-8caa-7afae8cc707c"
-					(reference "TP5")
-					(unit 1)
-				)
-			)
-		)
-	)
-	(wire
-		(pts
-			(xy 379.73 190.5)
-			(xy 379.73 193.04)
-		)
-		(stroke
-			(width 0)
-			(type default)
-		)
-	)
-	(label "TXD0"
-		(at 379.73 193.04 270)
-		(fields_autoplaced yes)
-		(effects
-			(font
-				(size 1.27 1.27)
-			)
-			(justify right bottom)
-		)
-	)
-	(symbol
-		(lib_id "Connector:TestPoint")
-		(at 397.51 190.5 0)
-		(unit 1)
-		(exclude_from_sim no)
-		(in_bom yes)
-		(on_board yes)
-		(dnp no)
-		(property "Reference" "TP6"
-			(at 397.51 186.69 0)
-			(effects
-				(font
-					(size 1.27 1.27)
-				)
-			)
-		)
-		(property "Value" "RXD0"
-			(at 397.51 194.31 0)
-			(effects
-				(font
-					(size 1.27 1.27)
-				)
-			)
-		)
-		(property "Footprint" "TestPoint:TestPoint_Pad_1.5x1.5mm"
-			(at 397.51 190.5 0)
-			(effects
-				(font
-					(size 1.27 1.27)
-				)
-				(hide yes)
-			)
-		)
-		(property "Datasheet" "~"
-			(at 397.51 190.5 0)
-			(effects
-				(font
-					(size 1.27 1.27)
-				)
-				(hide yes)
-			)
-		)
-		(property "Description" "Test pad 1.5 mm"
-			(at 397.51 190.5 0)
-			(effects
-				(font
-					(size 1.27 1.27)
-				)
-				(hide yes)
-			)
-		)
-		(property "LCSC" ""
-			(at 397.51 190.5 0)
-			(effects
-				(font
-					(size 1.27 1.27)
-				)
-				(hide yes)
-			)
-		)
-		(pin "1"
-		)
-		(instances
-			(project "pl60c_dmx_mini"
-				(path "/e63f84e3-7254-5f79-8caa-7afae8cc707c"
-					(reference "TP6")
-					(unit 1)
-				)
-			)
-		)
-	)
-	(wire
-		(pts
-			(xy 397.51 190.5)
-			(xy 397.51 193.04)
-		)
-		(stroke
-			(width 0)
-			(type default)
-		)
-	)
-	(label "RXD0"
-		(at 397.51 193.04 270)
-		(fields_autoplaced yes)
-		(effects
-			(font
-				(size 1.27 1.27)
-			)
-			(justify right bottom)
-		)
-	)
 	(wire
 		(pts
@@
 		)
 	)
-	(text "Test pads: I2C expansion and UART0"
+	(text "Test pads: I2C expansion (RTC / sensor)"
 		(exclude_from_sim no)
 		(at 272 165 0)
