File: pcb/pl60c_dmx.kicad_sch (KiCad schematic)
At the start: 39 parts, among them J1 USB-C 16P, J2 XLR-5 female (DMX OUT), J3 DMX pigtail, J4 EXPANSION, J5 UART0, Q1 S8050, SW1 RESET, SW2 BOOT, SW3 USER, U1 ESP32-S3-WROOM-1-N8, U2 AMS1117-3.3, U3 MAX3485, U4 USBLC6-2SC6

Commit message: auto: 2026-09-02 13:04:43
Co-Authored-By: Claude Fable 5.1 <noreply@anthropic.com>
Claude-Session: https://claude.ai/code/session_01WsrVZb94LwbHVAmBvsSTfn
Parts:
- D1: value SM712 -> PSM712; LCSC C58274 -> C32677; MPN SM712 -> PSM712-LF-T7
- D3: value 1N4148W -> B5819W; symbol Diode:1N4148W -> Device:D_Schottky; LCSC C81598 -> C8598; MPN (none) -> B5819W SL
- F1: value 0.75A PTC -> 1A PTC; LCSC C70069 -> C5358568; MPN (none) -> BSMD1206-100-30V
- J2: symbol Connector_Audio:XLR5 -> Connector_Audio:XLR5_Ground; LCSC (none) -> C368501
- J3: footprint TerminalBlock:TerminalBlock_bornier-3_P5.08mm -> TerminalBlock_Phoenix:TerminalBlock_Phoenix_MKDS-1,5-3-5.08_1x03_P5.08mm_Horizontal; LCSC C474881 -> C474953; MPN KF301-5.0-3P -> KF128-5.08-3P-AA
- J4: LCSC C2337 -> C37208; MPN (none) -> 2.54-1x6P
- J5: LCSC C2337 -> C124378; MPN (none) -> B-2100S04P-A110
- R1, R2: LCSC C25905 -> C23186
- SW1, SW2, SW3: footprint Button_Switch_SMD:SW_SPST_PTS645Sx43SMTR92 -> Button_Switch_SMD:SW_SPST_SKQG_WithStem; MPN (none) -> TS-1187A-B-A-B
- U1: value ESP32-S3-WROOM-1-N8 -> ESP32-S3-WROOM-1-N16R8; MPN ESP32-S3-WROOM-1-N8 -> ESP32-S3-WROOM-1-N16R8
- U3: value MAX3485 -> SP3485EN; symbol Interface_UART:MAX3485 -> Interface_UART:SP3485EN; LCSC C6785 -> C8963; MPN MAX3485ESA+T -> SP3485EN-L/TR
Connections:
- no-connect marks 26 -> 27
Changed lines of the file:
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@@
 			)
 		)
-		(property "LCSC" "C25905"
+		(property "LCSC" "C23186"
 			(at 74.93 80.01 0)
 			(effects
@@
 			)
 		)
-		(property "LCSC" "C25905"
+		(property "LCSC" "C23186"
 			(at 85.09 80.01 0)
 			(effects
@@
 			)
 		)
-		(property "Value" "0.75A PTC"
+		(property "Value" "1A PTC"
 			(at 69.85 46.99 0)
 			(effects
@@
 			)
 		)
-		(property "Description" "PTC resettable fuse 1206, 0.75 A hold"
+		(property "Description" "PTC resettable fuse 1206, 1 A hold / 1.8 A trip, 30 V"
 			(at 69.85 39.37 0)
 			(effects
@@
 			)
 		)
-		(property "LCSC" "C70069"
+		(property "LCSC" "C5358568"
+			(at 69.85 39.37 0)
+			(effects
+				(font
+					(size 1.27 1.27)
+				)
+				(hide yes)
+			)
+		)
+		(property "MPN" "BSMD1206-100-30V"
 			(at 69.85 39.37 0)
 			(effects
@@
 			)
 		)
-		(property "Value" "ESP32-S3-WROOM-1-N8"
+		(property "Value" "ESP32-S3-WROOM-1-N16R8"
 			(at 199.39 111.76 0)
 			(effects
@@
 			)
 		)
-		(property "Description" "ESP32-S3 WiFi/BLE module, 8 MB flash, PCB antenna"
+		(property "Description" "ESP32-S3 WiFi/BLE module, 16 MB flash + 8 MB PSRAM, PCB antenna"
 			(at 199.39 80.01 0)
 			(effects
@@
 			)
 		)
-		(property "MPN" "ESP32-S3-WROOM-1-N8"
+		(property "MPN" "ESP32-S3-WROOM-1-N16R8"
 			(at 199.39 80.01 0)
 			(effects
@@
 			)
 		)
-		(property "Footprint" "Button_Switch_SMD:SW_SPST_PTS645Sx43SMTR92"
+		(property "Footprint" "Button_Switch_SMD:SW_SPST_SKQG_WithStem"
 			(at 149.86 90.17 0)
 			(effects
@@
 			)
 		)
-		(property "Description" "Tactile switch 6x6 SMD"
+		(property "Description" "Tactile switch 5.1x5.1x1.5 mm SMD"
 			(at 149.86 90.17 0)
 			(effects
@@
 			)
 		)
+		(property "MPN" "TS-1187A-B-A-B"
+			(at 149.86 90.17 0)
+			(effects
+				(font
+					(size 1.27 1.27)
+				)
+				(hide yes)
+			)
+		)
 		(pin "1"
 		)
@@
 			)
 		)
-		(property "Footprint" "Button_Switch_SMD:SW_SPST_PTS645Sx43SMTR92"
+		(property "Footprint" "Button_Switch_SMD:SW_SPST_SKQG_WithStem"
 			(at 149.86 129.54 0)
 			(effects
@@
 			)
 		)
-		(property "Description" "Tactile switch 6x6 SMD"
+		(property "Description" "Tactile switch 5.1x5.1x1.5 mm SMD"
 			(at 149.86 129.54 0)
 			(effects
@@
 			)
 		)
+		(property "MPN" "TS-1187A-B-A-B"
+			(at 149.86 129.54 0)
+			(effects
+				(font
+					(size 1.27 1.27)
+				)
+				(hide yes)
+			)
+		)
 		(pin "1"
 		)
@@
 	)
 	(symbol
-		(lib_id "Interface_UART:MAX3485")
+		(lib_id "Interface_UART:SP3485EN")
 		(at 299.72 59.69 0)
 		(unit 1)
@@
 			)
 		)
-		(property "Value" "MAX3485"
+		(property "Value" "SP3485EN"
 			(at 299.72 78.74 0)
 			(effects
@@
 			)
 		)
-		(property "Description" "RS-485 transceiver 3.3V half-duplex SOIC-8"
+		(property "Description" "RS-485 transceiver 3.3 V half-duplex SOIC-8 (MAX3485 pin-compatible)"
 			(at 299.72 59.69 0)
 			(effects
@@
 			)
 		)
-		(property "LCSC" "C6785"
+		(property "LCSC" "C8963"
 			(at 299.72 59.69 0)
 			(effects
@@
 			)
 		)
-		(property "MPN" "MAX3485ESA+T"
+		(property "MPN" "SP3485EN-L/TR"
 			(at 299.72 59.69 0)
 			(effects
@@
 			)
 		)
-		(property "Value" "SM712"
+		(property "Value" "PSM712"
 			(at 330.2 97.79 0)
 			(effects
@@
 			)
 		)
-		(property "Description" "RS-485 TVS array +12/-7V SOT-23"
+		(property "Description" "RS-485 TVS array +12/-7 V 600 W SOT-23"
 			(at 330.2 90.17 0)
 			(effects
@@
 			)
 		)
-		(property "LCSC" "C58274"
+		(property "LCSC" "C32677"
 			(at 330.2 90.17 0)
 			(effects
@@
 			)
 		)
-		(property "MPN" "SM712"
+		(property "MPN" "PSM712-LF-T7"
 			(at 330.2 90.17 0)
 			(effects
@@
 	)
 	(symbol
-		(lib_id "Connector_Audio:XLR5")
+		(lib_id "Connector_Audio:XLR5_Ground")
 		(at 384.81 59.69 0)
 		(unit 1)
@@
 			)
 		)
-		(property "Description" "XLR 5-pin female, horizontal PCB mount (DMX OUT)"
+		(property "Description" "Neutrik XLR 5-pin female, horizontal PCB mount (DMX OUT)"
 			(at 384.81 59.69 0)
 			(effects
@@
 			)
 		)
-		(property "LCSC" ""
+		(property "LCSC" "C368501"
 			(at 384.81 59.69 0)
 			(effects
@@
 		(pin "5"
 		)
+		(pin "G"
+		)
 		(instances
 			(project "pl60c_dmx"
@@
 		(at 392.43 59.69)
 	)
+	(no_connect
+		(at 382.27 67.31)
+	)
 	(symbol
 		(lib_id "Connector:Screw_Terminal_01x03")
@@
 			)
 		)
-		(property "Footprint" "TerminalBlock:TerminalBlock_bornier-3_P5.08mm"
+		(property "Footprint" "TerminalBlock_Phoenix:TerminalBlock_Phoenix_MKDS-1,5-3-5.08_1x03_P5.08mm_Horizontal"
 			(at 384.81 95.25 0)
 			(effects
@@
 			)
 		)
-		(property "LCSC" "C474881"
+		(property "LCSC" "C474953"
 			(at 384.81 95.25 0)
 			(effects
@@
 			)
 		)
-		(property "MPN" "KF301-5.0-3P"
+		(property "MPN" "KF128-5.08-3P-AA"
 			(at 384.81 95.25 0)
 			(effects
@@
 			)
 		)
-		(property "Footprint" "Button_Switch_SMD:SW_SPST_PTS645Sx43SMTR92"
+		(property "Footprint" "Button_Switch_SMD:SW_SPST_SKQG_WithStem"
 			(at 199.39 214.63 0)
 			(effects
@@
 			)
 		)
-		(property "Description" "Tactile switch 6x6 SMD (snooze / manual on)"
+		(property "Description" "Tactile switch 5.1x5.1x1.5 mm SMD (snooze / manual on)"
 			(at 199.39 214.63 0)
 			(effects
@@
 			)
 		)
+		(property "MPN" "TS-1187A-B-A-B"
+			(at 199.39 214.63 0)
+			(effects
+				(font
+					(size 1.27 1.27)
+				)
+				(hide yes)
+			)
+		)
 		(pin "1"
 		)
@@
 	)
 	(symbol
-		(lib_id "Diode:1N4148W")
+		(lib_id "Device:D_Schottky")
 		(at 255.27 224.79 90)
 		(unit 1)
@@
 			)
 		)
-		(property "Value" "1N4148W"
+		(property "Value" "B5819W"
 			(at 255.27 228.6 0)
 			(effects
@@
 			)
 		)
-		(property "Description" "Flyback diode SOD-123"
+		(property "Description" "Schottky flyback diode 1 A 40 V SOD-123"
 			(at 255.27 224.79 0)
 			(effects
@@
 			)
 		)
-		(property "LCSC" "C81598"
+		(property "LCSC" "C8598"
+			(at 255.27 224.79 0)
+			(effects
+				(font
+					(size 1.27 1.27)
+				)
+				(hide yes)
+			)
+		)
+		(property "MPN" "B5819W SL"
 			(at 255.27 224.79 0)
 			(effects
@@
 			)
 		)
-		(property "Description" "Magnetic buzzer 8.5 mm SMD, 3-5 V, passive (drive with PWM ~2.7 kHz)"
+		(property "Description" "Magnetic buzzer 8.5x8.5 mm SMD, passive, 16 ohm, drive 2.7 kHz square wave"
 			(at 245.11 199.39 0)
 			(effects
@@
 			)
 		)
-		(property "LCSC" "C2337"
+		(property "LCSC" "C37208"
+			(at 299.72 190.5 0)
+			(effects
+				(font
+					(size 1.27 1.27)
+				)
+				(hide yes)
+			)
+		)
+		(property "MPN" "2.54-1x6P"
 			(at 299.72 190.5 0)
 			(effects
@@
 			)
 		)
-		(property "LCSC" "C2337"
+		(property "LCSC" "C124378"
+			(at 359.41 190.5 0)
+			(effects
+				(font
+					(size 1.27 1.27)
+				)
+				(hide yes)
+			)
+		)
+		(property "MPN" "B-2100S04P-A110"
 			(at 359.41 190.5 0)
 			(effects

Commit message: auto: 2026-09-02 13:06:45
Co-Authored-By: Claude Fable 5.1 <noreply@anthropic.com>
Claude-Session: https://claude.ai/code/session_01WsrVZb94LwbHVAmBvsSTfn
Parts:
- C6: footprint Capacitor_SMD:C_0603_1608Metric -> Capacitor_SMD:C_0805_2012Metric; LCSC C15849 -> C28323; MPN (none) -> CL21B105KBFNNNE
Changed lines of the file:
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@@
 			)
 		)
-		(property "Footprint" "Capacitor_SMD:C_0603_1608Metric"
+		(property "Footprint" "Capacitor_SMD:C_0805_2012Metric"
 			(at 157.48 77.47 0)
 			(effects
@@
 			)
 		)
-		(property "Description" "1uF 50V X7R 0603"
+		(property "Description" "1uF 50V X7R 0805 (EN reset delay)"
 			(at 157.48 77.47 0)
 			(effects
@@
 			)
 		)
-		(property "LCSC" "C15849"
+		(property "LCSC" "C28323"
 			(at 157.48 77.47 0)
 			(effects
+				(font
+					(size 1.27 1.27)
+				)
+				(hide yes)
+			)
+		)
+		(property "MPN" "CL21B105KBFNNNE"
+			(at 157.48 77.47 0)
+			(effects

Commit message: auto: 2026-09-02 13:23:01
Co-Authored-By: Claude Fable 5.1 <noreply@anthropic.com>
Claude-Session: https://claude.ai/code/session_01WsrVZb94LwbHVAmBvsSTfn
Other:
- moved on the sheet: D3, F1, R8, R9
Changed lines of the file:
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@@
 	(symbol
 		(lib_id "Device:Polyfuse")
-		(at 69.85 39.37 90)
+		(at 69.85 39.37 0)
 		(unit 1)
 		(exclude_from_sim no)
@@
 	(wire
 		(pts
-			(xy 66.04 39.37)
-			(xy 63.5 39.37)
+			(xy 69.85 35.56)
+			(xy 69.85 33.02)
 		)
 		(stroke
@@
 	)
 	(label "VBUS"
-		(at 63.5 39.37 180)
+		(at 69.85 33.02 90)
 		(fields_autoplaced yes)
 		(effects
@@
 				(size 1.27 1.27)
 			)
-			(justify right bottom)
+			(justify left bottom)
 		)
 	)
 	(wire
 		(pts
-			(xy 73.66 39.37)
-			(xy 76.2 39.37)
+			(xy 69.85 43.18)
+			(xy 69.85 45.72)
 		)
 		(stroke
@@
 	)
 	(label "+5V"
-		(at 76.2 39.37 0)
+		(at 69.85 45.72 270)
 		(fields_autoplaced yes)
 		(effects
@@
 				(size 1.27 1.27)
 			)
-			(justify left bottom)
+			(justify right bottom)
 		)
 	)
@@
 	(symbol
 		(lib_id "Device:R")
-		(at 144.78 209.55 90)
+		(at 144.78 214.63 0)
 		(unit 1)
 		(exclude_from_sim no)
@@
 		(dnp no)
 		(property "Reference" "R8"
-			(at 144.78 201.93 0)
+			(at 144.78 207.01 0)
 			(effects
 				(font
@@
 		)
 		(property "Value" "330R"
-			(at 144.78 217.17 0)
+			(at 144.78 222.25 0)
 			(effects
 				(font
@@
 		)
 		(property "Footprint" "Resistor_SMD:R_0603_1608Metric"
-			(at 144.78 209.55 0)
+			(at 144.78 214.63 0)
 			(effects
 				(font
@@
 		)
 		(property "Datasheet" "~"
-			(at 144.78 209.55 0)
+			(at 144.78 214.63 0)
 			(effects
 				(font
@@
 		)
 		(property "Description" "330R 0603 series (WS2812 data)"
-			(at 144.78 209.55 0)
+			(at 144.78 214.63 0)
 			(effects
 				(font
@@
 		)
 		(property "LCSC" "C23138"
-			(at 144.78 209.55 0)
+			(at 144.78 214.63 0)
 			(effects
 				(font
@@
 	(wire
 		(pts
-			(xy 140.97 209.55)
-			(xy 138.43 209.55)
+			(xy 144.78 210.82)
+			(xy 144.78 208.28)
 		)
 		(stroke
@@
 	)
 	(label "LED_DATA"
-		(at 138.43 209.55 180)
+		(at 144.78 208.28 90)
 		(fields_autoplaced yes)
 		(effects
@@
 				(size 1.27 1.27)
 			)
-			(justify right bottom)
+			(justify left bottom)
 		)
 	)
 	(wire
 		(pts
-			(xy 148.59 209.55)
-			(xy 151.13 209.55)
+			(xy 144.78 218.44)
+			(xy 144.78 220.98)
 		)
 		(stroke
@@
 	)
 	(label "LED_DATA_R"
-		(at 151.13 209.55 0)
+		(at 144.78 220.98 270)
 		(fields_autoplaced yes)
 		(effects
@@
 				(size 1.27 1.27)
 			)
-			(justify left bottom)
+			(justify right bottom)
 		)
 	)
@@
 	(symbol
 		(lib_id "Device:R")
-		(at 219.71 250.19 90)
+		(at 222.25 250.19 0)
 		(unit 1)
 		(exclude_from_sim no)
@@
 		(dnp no)
 		(property "Reference" "R9"
-			(at 219.71 242.57 0)
+			(at 222.25 242.57 0)
 			(effects
 				(font
@@
 		)
 		(property "Value" "1k"
-			(at 219.71 257.81 0)
+			(at 222.25 257.81 0)
 			(effects
 				(font
@@
 		)
 		(property "Footprint" "Resistor_SMD:R_0603_1608Metric"
-			(at 219.71 250.19 0)
+			(at 222.25 250.19 0)
 			(effects
 				(font
@@
 		)
 		(property "Datasheet" "~"
-			(at 219.71 250.19 0)
+			(at 222.25 250.19 0)
 			(effects
 				(font
@@
 		)
 		(property "Description" "1k 0603"
-			(at 219.71 250.19 0)
+			(at 222.25 250.19 0)
 			(effects
 				(font
@@
 		)
 		(property "LCSC" "C21190"
-			(at 219.71 250.19 0)
+			(at 222.25 250.19 0)
 			(effects
 				(font
@@
 	(wire
 		(pts
-			(xy 215.9 250.19)
-			(xy 213.36 250.19)
+			(xy 222.25 246.38)
+			(xy 222.25 243.84)
 		)
 		(stroke
@@
 	)
 	(label "BUZZER"
-		(at 213.36 250.19 180)
+		(at 222.25 243.84 90)
 		(fields_autoplaced yes)
 		(effects
@@
 				(size 1.27 1.27)
 			)
-			(justify right bottom)
+			(justify left bottom)
 		)
 	)
 	(wire
 		(pts
-			(xy 223.52 250.19)
-			(xy 226.06 250.19)
+			(xy 222.25 254)
+			(xy 222.25 256.54)
 		)
 		(stroke
@@
 	)
 	(label "Q1_B"
-		(at 226.06 250.19 0)
+		(at 222.25 256.54 270)
 		(fields_autoplaced yes)
 		(effects
@@
 				(size 1.27 1.27)
 			)
-			(justify left bottom)
+			(justify right bottom)
 		)
 	)
@@
 	(symbol
 		(lib_id "Device:D_Schottky")
-		(at 255.27 224.79 90)
+		(at 232.41 224.79 0)
 		(unit 1)
 		(exclude_from_sim no)
@@
 		(dnp no)
 		(property "Reference" "D3"
-			(at 255.27 220.98 0)
+			(at 232.41 220.98 0)
 			(effects
 				(font
@@
 		)
 		(property "Value" "B5819W"
-			(at 255.27 228.6 0)
+			(at 232.41 228.6 0)
 			(effects
 				(font
@@
 		)
 		(property "Footprint" "Diode_SMD:D_SOD-123"
-			(at 255.27 224.79 0)
+			(at 232.41 224.79 0)
 			(effects
 				(font
@@
 		)
 		(property "Datasheet" "~"
-			(at 255.27 224.79 0)
+			(at 232.41 224.79 0)
 			(effects
 				(font
@@
 		)
 		(property "Description" "Schottky flyback diode 1 A 40 V SOD-123"
-			(at 255.27 224.79 0)
+			(at 232.41 224.79 0)
 			(effects
 				(font
@@
 		)
 		(property "LCSC" "C8598"
-			(at 255.27 224.79 0)
+			(at 232.41 224.79 0)
 			(effects
 				(font
@@
 		)
 		(property "MPN" "B5819W SL"
-			(at 255.27 224.79 0)
+			(at 232.41 224.79 0)
 			(effects
 				(font
@@
 	(wire
 		(pts
-			(xy 255.27 228.6)
-			(xy 255.27 231.14)
+			(xy 228.6 224.79)
+			(xy 226.06 224.79)
 		)
 		(stroke
@@
 	)
 	(label "+5V"
-		(at 255.27 231.14 270)
+		(at 226.06 224.79 180)
 		(fields_autoplaced yes)
 		(effects
@@
 	(wire
 		(pts
-			(xy 255.27 220.98)
-			(xy 255.27 218.44)
+			(xy 236.22 224.79)
+			(xy 238.76 224.79)
 		)
 		(stroke
@@
 	)
 	(label "BZ_N"
-		(at 255.27 218.44 90)
+		(at 238.76 224.79 0)
 		(fields_autoplaced yes)
 		(effects
