File: pcb/pl60c_dmx.kicad_sch (KiCad schematic)
At the start: 39 parts, among them J1 USB-C 16P, J2 XLR-5 female (DMX OUT), J3 DMX pigtail, J4 EXPANSION, J5 UART0, Q1 S8050, SW1 RESET, SW2 BOOT, SW3 USER, U1 ESP32-S3-WROOM-1-N16R8, U2 AMS1117-3.3, U3 SP3485EN, U4 USBLC6-2SC6

Commit message: auto: 2026-09-02 14:48:00
Co-Authored-By: Claude Fable 5.1 <noreply@anthropic.com>
Claude-Session: https://claude.ai/code/session_01WsrVZb94LwbHVAmBvsSTfn
Parts:
- added R10: 10R, Resistor_SMD:R_1206_3216Metric, symbol Device:R
- C2: value 10uF -> 22uF; LCSC C15850 -> C45783
- D2: value WS2812B -> WS2812B-2020; footprint LED_SMD:LED_WS2812B_PLCC4_5.0x5.0mm_P3.2mm -> LED_SMD:LED_WS2812B-2020_PLCC4_2.0x2.0mm; symbol LED:WS2812B -> LED:WS2812B-2020; LCSC C2761795 -> C52917434; MPN WS2812B-B/T -> WS2812B-2020-V6
- Q1: symbol Transistor_BJT:S8050 -> Transistor_BJT:BC817
- R9: value 1k -> 470R; LCSC C21190 -> C23179
Connections:
- net +3V3: now also D2.4 (VDD); no longer D2.1 (VDD)
- net +5V: now also R10.1; no longer BZ1.1 (+), D3.1 (K)
- net GND: now also D2.2 (VSS), Q1.2 (E); no longer D2.3 (VSS), Q1.1 (E)
- net LED_DATA_R: now also D2.3 (DIN); no longer D2.4 (DIN)
- net Q1_B: now also Q1.1 (B); no longer Q1.2 (B)
- new net BZ_P: BZ1.1 (+), D3.1 (K), R10.2
